File: Design Files/V2I1/A2027.kicad_sch (KiCad schematic)
At the start: 83 parts, among them J1 Screw_Terminal_01x02, J2 USB_B_Micro, J3 Conn_02x03_Top_Bottom, J4 Conn_01x05_Pin, J5 DE9_Pins, J6 Conn_01x02_Pin, J7 Conn_01x04_Pin, Q1 BSS138, Q2 BC857, Q3 BSS138, Q4 BC857, SW1 SW_SPDT, U1 TPS560200, U2 USBLC6-2SC6, U3 TPS2113A, U4 STM32F103C8T6, U5 LM1117MP-3.3, U6 DS3232M, U7 MAX3232, U8 24LC256, Y1 16MHz

Commit message: master :: update schmea
Parts:
- BT1: footprint (none) -> Battery:BatteryHolder_Keystone_3034_1x20mm
- SW1: footprint Button_Switch_THT:SW_E-Switch_EG1224_SPDT_Angled -> Button_Switch_SMD:SW_SPDT_PCM12
- U3: footprint (none) -> Package_SO:TSSOP-8_4.4x3mm_P0.65mm
- U7: footprint (none) -> Package_SO:TSSOP-16_4.4x5mm_P0.65mm
Changed lines of the file:
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@@
 			)
 		)
-		(property "Footprint" ""
+		(property "Footprint" "Package_SO:TSSOP-8_4.4x3mm_P0.65mm"
 			(at 63.5 86.36 0)
 			(hide yes)
@@
 			)
 		)
-		(property "Footprint" ""
+		(property "Footprint" "Package_SO:TSSOP-16_4.4x5mm_P0.65mm"
 			(at 233.68 226.06 0)
 			(hide yes)
@@
 			)
 		)
-		(property "Footprint" "Button_Switch_THT:SW_E-Switch_EG1224_SPDT_Angled"
+		(property "Footprint" "Button_Switch_SMD:SW_SPDT_PCM12"
 			(at 228.6 59.69 0)
 			(hide yes)
@@
 		(property "Value" "Screw_Terminal_01x02"
 			(at 39.624 37.846 0)
+			(hide yes)
 			(show_name no)
 			(do_not_autoplace no)
@@
 			)
 		)
-		(property "Footprint" ""
+		(property "Footprint" "Battery:BatteryHolder_Keystone_3034_1x20mm"
 			(at 119.38 129.286 90)
 			(hide yes)

Commit message: placement
Parts:
- removed J3: Conn_02x03_Top_Bottom, Connector_PinHeader_2.54mm:PinHeader_2x03_P2.54mm_Vertical, symbol Connector_Generic:Conn_02x03_Top_Bottom
- removed J6: Conn_01x02_Pin, Connector_PinHeader_2.54mm:PinHeader_1x02_P2.54mm_Vertical, symbol Connector:Conn_01x02_Pin
- added D1: SS14, Diode_SMD:D_SMA, symbol Diode:SS14
- added J5: Conn_01x04_Pin, Connector_PinHeader_2.54mm:PinHeader_1x04_P2.54mm_Vertical, symbol Connector:Conn_01x04_Pin
- added JP1: SolderJumper_3_Open, Jumper:SolderJumper-3_P2.0mm_Open_TrianglePad1.0x1.5mm, symbol Jumper:SolderJumper_3_Open
- added R8: 10k, Resistor_SMD:R_0402_1005Metric, symbol Device:R
- J2: footprint (none) -> Connector_USB:USB_Micro-B_Wuerth_629105150521
- J4: renamed from J5; footprint (none) -> Connector_Dsub:DSUB-9_Pins_Horizontal_P2.77x2.84mm_EdgePinOffset7.70mm_Housed_MountingHolesOffset9.12mm
- renumbered D9 to D10, D10 to D11, D11 to D12, D1 to D2, D2 to D3, D3 to D4, D4 to D5, D5 to D6, D6 to D7, D7 to D8, D8 to D9, J4 to J3, J7 to J6, R9 to R10, R10 to R11, R11 to R12, R12 to R13, R13 to R14, R14 to R15, R15 to R16, R16 to R17, R17 to R18, R18 to R19, R19 to R20, R8 to R9
Connections:
- net +12V: now also D1.1 (K); no longer J1.1 (Pin_1)
- net +3.3V: now also J5.1 (Pin_1), JP1.3 (B)
- net E_USB_D+: now also U2.3 (I/O2); no longer U2.6 (I/O1)
- net E_USB_D-: now also U2.1 (I/O1); no longer U2.4 (I/O2)
- net GND: now also R3.2, J5.4 (Pin_4), JP1.1 (A)
- net I2C2_SCL: now also J5.2 (Pin_2)
- net I2C2_SDA: now also J5.3 (Pin_3)
- net USB_D+: now also U2.4 (I/O2); no longer U2.1 (I/O1)
- net USB_D-: now also U2.6 (I/O1); no longer U2.3 (I/O2)
- net at U4.20 (PB2): now also R8.2
- net at C6.2, R1.2, R2.1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: no longer R3.2
- net EEPROM_WP: no longer names the net of U8.7 (WP)
- net EEPROM_WP: no longer U4.12 (PA2)
- new net: JP1.2 (C), R8.1
- new net: D1.2 (A), J1.1 (Pin_1)
- no-connect marks 33 -> 40
Other:
- note added: "e.g. CR2032 battery cell"
- note removed: "e.g. CR2016 battery cell"
- moved on the sheet: U2

Commit message: master :: board outline
Parts:
- added H1: MountingHole, MountingHole:MountingHole_3.2mm_M3, symbol Mechanical:MountingHole
- added H2, H3, H4: MountingHole_Pad, MountingHole:MountingHole_3.2mm_M3_Pad_TopBottom, symbol Mechanical:MountingHole_Pad
Connections:
- net GND: now also H2.1, H3.1, H4.1
Other:
- note added: "M3"
- note added: "Mouting Holes"

Commit message: master :: routing
Parts:
- R6: footprint Resistor_SMD:R_0402_1005Metric -> Resistor_SMD:R_0603_1608Metric
Connections:
- net E_USB_D+: now also U2.6 (I/O1); no longer U2.3 (I/O2)
- net E_USB_D-: now also U2.4 (I/O2); no longer U2.1 (I/O1)
- net USB_D+: now also U2.1 (I/O1); no longer U2.4 (I/O2)
- net USB_D-: now also U2.3 (I/O2); no longer U2.6 (I/O1)
Other:
- moved on the sheet: U2

Commit message: master :: update
Connections:
- net BOOT1: now reaches R8.2, U4.20 (PB2)
- net SW_BOOT1: now reaches JP1.2 (C), R8.1
Changed lines of the file:
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@@
+		)
+	)
+	(label "BOOT1"
+		(at 259.08 87.63 0)
+		(effects
+			(font
+				(size 1.27 1.27)
+			)
+			(justify left bottom)
 		)
 	)
@@
 		(effects
 			(font
+				(size 1.27 1.27)
+			)
+			(justify left bottom)
+		)
+	)
+	(label "SW_BOOT1"
+		(at 243.84 95.25 0)
+		(effects
+			(font
